File: pandora13-wifi-controller_pcb/pandora13-wifi-controller_pcb.kicad_pcb (KiCad board)
At the start: 2 copper layers, 85.7 x 73 mm, 10 parts, among them J1 Screw_Terminal_01x02, J2 Screw_Terminal_01x02, J3 Screw_Terminal_01x02, J4 Screw_Terminal_01x02, J5 Screw_Terminal_01x02, J6 Screw_Terminal_01x02, J7 Screw_Terminal_01x02, U1 Pico, U2 ULN2003, U3 ULN2003

Commit message: Labels on back silkscreen for each of the buttons
Other:
- board text added: "GND left"
- board text added: "a b"
- board text added: "c d"
- board text added: "e f"
- board text added: "right start"
- board text added: "up down"
Changed lines of the file:
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@@
   (gr_rect (start 50.19 53.22) (end 135.91 126.26)
     (stroke (width 0.1) (type default)) (fill none) (layer "Edge.Cuts"))
+  (gr_text "e\n\nf" (at 53.96 85.84) (layer "B.SilkS")
+    (effects (font (size 1 1) (thickness 0.15)) (justify left bottom mirror))
+  )
+  (gr_text "up\n\n\ndown" (at 56.93 96.95) (layer "B.SilkS")
+    (effects (font (size 1 1) (thickness 0.15)) (justify left bottom mirror))
+  )
+  (gr_text "GND\n\n\nleft" (at 58.3 108.81) (layer "B.SilkS")
+    (effects (font (size 1 1) (thickness 0.15)) (justify left bottom mirror))
+  )
+  (gr_text "a\n\nb" (at 54.38 61.84) (layer "B.SilkS")
+    (effects (font (size 1 1) (thickness 0.15)) (justify left bottom mirror))
+  )
+  (gr_text "c\n\nd" (at 54.13 74.14) (layer "B.SilkS")
+    (effects (font (size 1 1) (thickness 0.15)) (justify left bottom mirror))
+  )
+  (gr_text "right\n\n\nstart" (at 57.49 120.76) (layer "B.SilkS")
+    (effects (font (size 1 1) (thickness 0.15)) (justify left bottom mirror))
+  )
   (gr_text "PANDORA13 WIFI CONTROLLER\n2024-01-07" (at 88.85 121.89) (layer "F.SilkS")
     (effects (font (size 1 1) (thickness 0.15)) (justify left bottom))
